File: CAD/Barone2_Eagle_CAD/v1.9.brd (EAGLE design)
At the start: 101.6 x 101.6 mm, 57 parts, among them J1 USB_C_Port_Raspberry_Pi, J2 XT60-M, J3 10033854-052FSLF, M1 PIC32MX340F512H-80I/MR, M2 RaspberryPi_DDR2_SODIMM_1.8V, Q2 BSS138

Commit message: wiring up board
Parts:
- removed 2V8_OUT: STMICROELECTRONICS_LD1117DT33CTRSTMICROELECTRONICS_LD1117DT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, STMicroelectronics - LD1117DT33CTR:STMICROELECTRONICS_LD1117DT33CTR_2
- removed C10: 0.1uF, rcl:C0805
- removed C8: 10uF, rcl:C0805
- removed J3: 10033854-052FSLF, 10033854-052FSLF:AMPHENOL_10033854-052FSLF
- removed M2: RaspberryPi_DDR2_SODIMM_1.8V, con-amp:SLOT-1376408-1_1.8V
- added 1V8_OUT1: STMICROELECTRONICS_LD1117DT33CTRSTMICROELECTRONICS_LD1117DT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, STMicroelectronics - LD1117DT33CTR:STMICROELECTRONICS_LD1117DT33CTR_2
- added C20: 10uF, rcl:C0805
- added C21: 0.1uF, rcl:C0805
- added C22: 0.01uF, rcl:C0805
- added JP1: (no value), adafruit:1X08-CLEANBIG
- added Q1, SCL_OUT_IMU1: BSS138, BSS138:SOT95P240X111-3N
- added SODIMM_M2_PINOUT: 10033854-052FSLF, 10033854-052FSLF:AMPHENOL_10033854-052FSLF
- added X1: CB3LV-3C-8M0000, CB3LV-3C-20M0000:OSCCC700X500X180-4N
- added Y1: ABRACON_ASEK-32_768KHZ-LRTABRACON_ASEK-32_768KHZ-LRT_0_0, Abracon - ASEK-32.768KHZ-LRT:ABRACON_ASEK-32_768KHZ-LRT_0
- moved J2 110.1 mm to (6.35, 19.1), turned to 270 degrees
- moved U.FL 80.7 mm to (91.4, 14.0)
- moved D4 77.7 mm to (80.0, 38.1)
- moved C6 73.0 mm to (88.9, 87.6)
- moved 1V8_OUT 73.0 mm to (87.6, 95.2)
- moved C9 73.0 mm to (82.5, 87.6)
- moved GPS 72.7 mm to (83.8, 25.4)
- moved B1 59.8 mm to (71.1, 43.2)
- moved C5 55.9 mm to (16.5, 40.6), turned to 180 degrees
- moved U$6 43.2 mm to (83.8, 73.7)
- moved C11 35.1 mm to (15.2, 35.6)
- moved C17 34.9 mm to (11.4, 45.7)
- moved MPR 34.5 mm to (20.3, 35.6)
- moved R15 32.6 mm to (11.4, 48.3), turned to 180 degrees
- moved M1 31.8 mm to (19.1, 47.0)
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Connections:
- net +5V renamed 5V
- net N$1 renamed VCAP_VCORE_M1
- removed net 2.8V: 2V8_OUT.4, C8.1
- removed net D+_M2: J1.5, J1.8, M2.167
- removed net D-_M2: J1.6, J1.7, M2.165
- removed net M2_1V8: M2.183, M2.184, M2.185, M2.186
- removed net M2_VBAT: M2.197, M2.198, M2.199, M2.200
- removed net MISO_M1: M1.12, M2.29, R1.2, U$6.7
- removed net MOSI_M1: M1.11, M2.33, R11.2, U$6.3
- removed net N$15: M2.41, M2.42
- removed net SCK_M1: M1.13, M2.35, R12.2, U$6.5
- new net AVDD3_M1: C16.2, M1.38
- new net AVDD_M1: C5.2, M1.19
- new net AVSS_M1: C5.1, M1.20
- new net GPIO13_M2: JP1.8, SODIMM_M2_PINOUT.47
- new net GPIO14_M2: JP1.7, SODIMM_M2_PINOUT.51
- new net GPIO15_M2: JP1.6, SODIMM_M2_PINOUT.53
- new net GPIO16_M2: JP1.5, SODIMM_M2_PINOUT.57
- new net GPIO17_M2: JP1.4, SODIMM_M2_PINOUT.59
- new net GPIO18_M2: JP1.3, SODIMM_M2_PINOUT.63
- new net GPIO19_M2: JP1.2, SODIMM_M2_PINOUT.65
- new net GPIO20_M2: JP1.1, SODIMM_M2_PINOUT.69
- new net IMU_SDA: IMU.24, Q1.3, SCL_OUT_IMU1.1
- new net MISO_M2: M1.12, R1.2, SODIMM_M2_PINOUT.29, U$6.7
- new net MOSI_M2: M1.11, R11.2, SODIMM_M2_PINOUT.33, U$6.3
- new net N$1: GPS.P$1
- new net N$4: R7.2
- new net N$6: M1.40, X1.1
- new net N$7: M1.39, X1.3
- new net N$8: M1.48, Y1.1
- new net SCK_M2: M1.13, R12.2, SODIMM_M2_PINOUT.35, U$6.5
- new net USB_D+_M2: J1.6, J1.7, SODIMM_M2_PINOUT.165
- new net USB_D-_M2: J1.5, J1.8, SODIMM_M2_PINOUT.167
- new net VDD1_M1: C17.2, M1.10
- new net VSS1_M1: C17.1, M1.9
- new net VSS3_M1: C16.1, M1.41
- net 1.8V: now also 1V8_OUT1.4, C14.1, C20.1, IMU.13, IMU.8, Q1.2, Q2.2, SODIMM_M2_PINOUT.183, SODIMM_M2_PINOUT.184, SODIMM_M2_PINOUT.185, SODIMM_M2_PINOUT.186
- net 9.6V-12.6V: no longer 1V8_OUT.3, 2V8_OUT.3, 5V_OUT.3, C10.1, C4.1, C9.1
- net CS_M1: now also SODIMM_M2_PINOUT.4, SODIMM_M2_PINOUT.5; no longer J3.5, M2.5
- net CS_MICRO_SD: now also SODIMM_M2_PINOUT.2; no longer J3.2, M2.3
- net GND: now also 1V8_OUT1.1, C20.2, C21.2, C22.2, SODIMM_M2_PINOUT.103, SODIMM_M2_PINOUT.104, SODIMM_M2_PINOUT.109, SODIMM_M2_PINOUT.110, SODIMM_M2_PINOUT.115, SODIMM_M2_PINOUT.116, SODIMM_M2_PINOUT.121, SODIMM_M2_PINOUT.122, SODIMM_M2_PINOUT.127, SODIMM_M2_PINOUT.133, SODIMM_M2_PINOUT.134, SODIMM_M2_PINOUT.139, SODIMM_M2_PINOUT.140, SODIMM_M2_PINOUT.145, SODIMM_M2_PINOUT.146, SODIMM_M2_PINOUT.151, SODIMM_M2_PINOUT.152, SODIMM_M2_PINOUT.157, SODIMM_M2_PINOUT.163, SODIMM_M2_PINOUT.164, SODIMM_M2_PINOUT.168, SODIMM_M2_PINOUT.169, SODIMM_M2_PINOUT.170, SODIMM_M2_PINOUT.181, SODIMM_M2_PINOUT.182, SODIMM_M2_PINOUT.187, SODIMM_M2_PINOUT.188, SODIMM_M2_PINOUT.19, SODIMM_M2_PINOUT.195, SODIMM_M2_PINOUT.196, SODIMM_M2_PINOUT.20, SODIMM_M2_PINOUT.31, SODIMM_M2_PINOUT.32, SODIMM_M2_PINOUT.37, SODIMM_M2_PINOUT.38, SODIMM_M2_PINOUT.43, SODIMM_M2_PINOUT.44, SODIMM_M2_PINOUT.49, SODIMM_M2_PINOUT.50, SODIMM_M2_PINOUT.55, SODIMM_M2_PINOUT.56, SODIMM_M2_PINOUT.61, SODIMM_M2_PINOUT.62, SODIMM_M2_PINOUT.67, SODIMM_M2_PINOUT.68, SODIMM_M2_PINOUT.7, SODIMM_M2_PINOUT.73, SODIMM_M2_PINOUT.74, SODIMM_M2_PINOUT.79, SODIMM_M2_PINOUT.8, SODIMM_M2_PINOUT.80, SODIMM_M2_PINOUT.85, SODIMM_M2_PINOUT.86, SODIMM_M2_PINOUT.91, SODIMM_M2_PINOUT.92, SODIMM_M2_PINOUT.97, SODIMM_M2_PINOUT.98, SODIMM_M2_PINOUT.S1, SODIMM_M2_PINOUT.S2, X1.2, Y1.2; no longer 2V8_OUT.1, C10.2, C16.1, C17.1, C5.1, C8.2, J3.7, J3.8, M1.20, M1.41, M1.9, M2.1, M2.103, M2.104, M2.109, M2.110, M2.115, M2.116, M2.121, M2.122, M2.127, M2.13, M2.133, M2.134, M2.139, M2.14, M2.140, M2.145, M2.146, M2.151, M2.152, M2.157, M2.163, M2.164, M2.168, M2.169, M2.170, M2.181, M2.182, M2.187, M2.188, M2.19, M2.195, M2.196, M2.20, M2.25, M2.26, M2.31, M2.32, M2.37, M2.38, M2.43, M2.44, M2.49, M2.50, M2.55, M2.56, M2.61, M2.62, M2.67, M2.68, M2.7, M2.73, M2.74, M2.79, M2.8, M2.80, M2.85, M2.86, M2.91, M2.92, M2.97, M2.98
- net GPIO12_M2: now also SODIMM_M2_PINOUT.45; no longer M2.45
- net GPIO2_M2: now also SODIMM_M2_PINOUT.9; no longer M2.9
- net GPIO3_M2: now also SODIMM_M2_PINOUT.11; no longer M2.11
- net GPIO4_M2: now also SODIMM_M2_PINOUT.15; no longer M2.15
- net GPIO5_M2: now also SODIMM_M2_PINOUT.17; no longer M2.17
- net GPIO6_M2: now also SODIMM_M2_PINOUT.21; no longer M2.21
- net GPIO7_M2: now also SODIMM_M2_PINOUT.23; no longer M2.23
- net GPIO8_M2: now also SODIMM_M2_PINOUT.27; no longer M2.27
- net N$9: now also M1.47, Y1.3; no longer M2.39, M2.40
- net SDA_M1: now also Q1.1, SCL_OUT_IMU1.3; no longer IMU.24
- net VIN: now also 1V8_OUT.3, 1V8_OUT1.3, 5V_OUT.3, C21.1, C22.1, C4.1, C9.1, SCL_OUT_IMU1.2, SODIMM_M2_PINOUT.189, SODIMM_M2_PINOUT.190, SODIMM_M2_PINOUT.191, SODIMM_M2_PINOUT.192, SODIMM_M2_PINOUT.193, SODIMM_M2_PINOUT.194, SODIMM_M2_PINOUT.197, SODIMM_M2_PINOUT.198, SODIMM_M2_PINOUT.199, SODIMM_M2_PINOUT.200, SODIMM_M2_PINOUT.39, SODIMM_M2_PINOUT.40, SODIMM_M2_PINOUT.41, SODIMM_M2_PINOUT.42, X1.4, Y1.4; no longer C14.1, C16.2, C17.2, C5.2, GPS.P$1, IMU.13, IMU.8, M1.10, M1.19, M1.38, M2.189, M2.190, M2.191, M2.193, Q2.2, R7.2
Routing:
- net 1.8V: track 0.00 -> 86.0 mm
- net VIN: track 3.56 -> 62.5 mm, vias 0 -> 15
- net 5V: track 0.00 -> 56.3 mm, vias 0 -> 1
- net MOSI_M2: track 0.00 -> 29.4 mm, vias 0 -> 2
- net GPIO8_M2: track 0.00 -> 26.0 mm, vias 0 -> 2
- net GPIO7_M2: track 0.00 -> 24.7 mm, vias 0 -> 2
- net GPIO6_M2: track 0.00 -> 23.1 mm, vias 0 -> 2
- net GPIO5_M2: track 0.00 -> 21.8 mm, vias 0 -> 2
- net GPIO12_M2: track 0.00 -> 20.4 mm, vias 0 -> 2
- net GPIO4_M2: track 0.00 -> 20.3 mm, vias 0 -> 2
- net GPIO3_M2: track 0.00 -> 19.0 mm, vias 0 -> 2
- net GPIO2_M2: track 0.00 -> 18.2 mm, vias 0 -> 2
- net 3.3V: track 0.00 -> 14.9 mm, vias 0 -> 2
- net SCK_M2: track 0.00 -> 14.3 mm
- net 9.6V-12.6V: track 0.00 -> 13.6 mm
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