File: CAD/Barone2_Eagle_CAD/v1.9.sch (EAGLE design)
At the start: 71 parts, among them J2 XT60-M, M1 PIC32MX340F512H-80I/MR, U1 FT232RQ, X1 CB3LV-3C-8M0000, Y1 ABRACON_ASEK-32_768KHZ-LRTABR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

Commit message: v1.9 finalized and sent to board house OSH Park
Parts:
- removed R12, R13, R14: 47k, adafruit:R-US_R0805W
Connections:
- removed net AVDD3_M1: C16.2, M1.VDD3
- removed net AVDD_M1: C5.2, M1.AVDD
- removed net AVSS_M1: C5.1, M1.AVSS
- removed net CS_M1: M1.AN2/C2IN-/!SS1!/CN4/RB2
- removed net VDD1_M1: C17.2, M1.VDD1
- removed net VDD2_M1: C15.2, ICSP.2, M1.VDD2
- removed net VSS1_M1: C17.1, M1.VSS1
- removed net VSS2_M1: C15.1, ICSP.3, M1.VSS2
- removed net VSS3_M1: C16.1, M1.VSS3
- net GND: now also C15.1, C16.1, C17.1, C5.1, ICSP.3, M1.AN2/C2IN-/!SS1!/CN4/RB2, M1.AVSS, M1.VSS1, M1.VSS2, M1.VSS3
- net MISO_M2: no longer R12.2
- net MOSI_M2: no longer R13.2
- net SCK_M2: no longer R14.2
- net VIN: now also C15.2, C16.2, C17.2, C5.2, ICSP.2, M1.AVDD, M1.VDD1, M1.VDD2, M1.VDD3; no longer R12.1, R13.1, R14.1
Other:
- moved on the sheet: C15, C16, C17, C5
